Commit message: enable realsense camera

File: husky_description/urdf/accessories/intel_realsense.urdf.xacro (robot description, xacro)
@@ -84,5 +84,6 @@
     </link>
     <joint type="fixed" name="${prefix}_realsense_lens_joint">
-      <origin xyz="0 0 0" rpy="0 0 0" />
+      <!-- Offset the camera 35cm forwards and 1cm up -->
+      <origin xyz="0.35 0 0.01" rpy="0 0 0" />
       <parent link="${parent_link}" />
       <child link="${prefix}_realsense_lens" />

File: husky_description/urdf/husky.urdf.xacro (robot description, xacro)
@@ -70,5 +70,5 @@
   <xacro:arg name="laser_3d_secondary_rpy"        default="$(optenv HUSKY_LASER_3D_SECONDARY_RPY 0 0 -3.14159)" />
   <!-- Realsense Camera Primary and Secondary -->
-  <xacro:arg name="realsense_enabled"             default="$(optenv HUSKY_REALSENSE_ENABLED 0)" />
+  <xacro:arg name="realsense_enabled"             default="$(optenv HUSKY_REALSENSE_ENABLED 1)" />
   <xacro:arg name="realsense_topic"               default="$(optenv HUSKY_REALSENSE_TOPIC realsense)" />
   <xacro:arg name="realsense_prefix"              default="$(optenv HUSKY_REALSENSE_PREFIX camera)" />
